File: box.kicad_pcb (KiCad board)
At the start: 2 copper layers, 112 x 36.6 mm, 42 parts, among them J1 Conn_01x03, J10 Conn_01x03, J11 Conn_01x05, J2 Conn_01x03, J3 Conn_01x03, J4 Conn_01x03, J5 Conn_01x03, J6 Conn_01x03, J7 Conn_01x03, J8 Conn_01x03, J9 Conn_01x03

Commit message: C7->D7
Other:
- board text added: "D3 D2 GND GND D1 D0 D4 C6 D7 E6 B4 B5"
- board text removed: "D3 D2 GND GND D1 D0 D4 C6 C7 E6 B4 B5"
Changed lines of the file:
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@@
     (effects (font (size 1.6 1.6) (thickness 0.15)) (justify left))
   )
-  (gr_text "D3\nD2\nGND\nGND\nD1\nD0\nD4\nC6\nC7\nE6\nB4\nB5" (at 104.902 118.872 90) (layer F.SilkS)
+  (gr_text "D3\nD2\nGND\nGND\nD1\nD0\nD4\nC6\nD7\nE6\nB4\nB5" (at 104.902 118.872 90) (layer F.SilkS)
     (effects (font (size 1.6 1.6) (thickness 0.15)) (justify right))
   )

Commit message: Update March 21st
Parts:
- removed C1, C2, C3, C4: 470n, Capacitor_SMD:C_0805_2012Metric_Pad1.15x1.40mm_HandSolder
- removed CT1: Conn_02x08_Counter_Clockwise, Connector_PinSocket_2.54mm:PinSocket_2x08_P2.54mm_Vertical
- removed H1, H2, H3: MountingHole_Pad, MountingHole:MountingHole_3.2mm_M3_DIN965_Pad
- removed J1, J10, J2, J3, J4, J5, J6, J7, J8, J9: Conn_01x03, Connector_PinSocket_2.54mm:PinSocket_1x03_P2.54mm_Vertical
- removed J11: Conn_01x05, Connector_PinSocket_2.54mm:PinSocket_1x05_P2.54mm_Vertical
- removed PM1: Pro_Micro, buttonbox:promicro
- removed R1, R10, R11, R12, R13, R14, R15, R16, R17, R18, R19, R2, R20, R3, R4, R5, R6, R7, R8, R9: 10k, Resistor_SMD:R_0805_2012Metric_Pad1.15x1.40mm_HandSolder
- removed SR1, SR2: Conn_02x08_Counter_Clockwise, Package_DIP:DIP-16_W7.62mm
- added B301: Conn_01x02, Connector_PinHeader_2.54mm:PinHeader_1x02_P2.54mm_Vertical, F.Cu at (225.5, 121.0)
- added B302: Conn_01x02, Connector_PinHeader_2.54mm:PinHeader_1x02_P2.54mm_Vertical, F.Cu at (225.5, 134.9)
- added B303: Conn_01x02, Connector_PinHeader_2.54mm:PinHeader_1x02_P2.54mm_Vertical, F.Cu at (225.5, 130.3)
- added B304: Conn_01x02, Connector_PinHeader_2.54mm:PinHeader_1x02_P2.54mm_Vertical, F.Cu at (225.5, 125.6)
- added B305: Conn_01x02, Connector_PinHeader_2.54mm:PinHeader_1x02_P2.54mm_Vertical, F.Cu at (232.7, 134.9)
- added B306: Conn_01x02, Connector_PinHeader_2.54mm:PinHeader_1x02_P2.54mm_Vertical, F.Cu at (232.7, 130.3)
- added B307: Conn_01x02, Connector_PinHeader_2.54mm:PinHeader_1x02_P2.54mm_Vertical, F.Cu at (232.7, 125.6)
- added B308: Conn_01x02, Connector_PinHeader_2.54mm:PinHeader_1x02_P2.54mm_Vertical, F.Cu at (239.9, 134.9)
- added C101: 470n, Capacitor_SMD:C_0805_2012Metric_Pad1.15x1.40mm_HandSolder, B.Cu at (96.8, 114.6)
- added C102: 470n, Capacitor_SMD:C_0805_2012Metric_Pad1.15x1.40mm_HandSolder, B.Cu at (106.8, 95.8)
- added C103: 470n, Capacitor_SMD:C_0805_2012Metric_Pad1.15x1.40mm_HandSolder, B.Cu at (106.6, 159.2)
- added C201: 470n, Capacitor_SMD:C_0805_2012Metric_Pad1.15x1.40mm_HandSolder, B.Cu at (129.3, 108.4)
- added C301: 470n, Capacitor_SMD:C_0805_2012Metric_Pad1.15x1.40mm_HandSolder, F.Cu at (173.4, 100.8)
- added H101: MountingHole_Pad, MountingHole:MountingHole_3.2mm_M3_DIN965_Pad, F.Cu at (75.2, 97.0)
- added H102: MountingHole_Pad, MountingHole:MountingHole_3.2mm_M3_DIN965_Pad, F.Cu at (213.9, 97.0)
- added H103: MountingHole_Pad, MountingHole:MountingHole_3.2mm_M3_DIN965_Pad, F.Cu at (73.2, 158.5)
- added H104: MountingHole_Pad, MountingHole:MountingHole_3.2mm_M3_DIN965_Pad, F.Cu at (213.4, 158.8)
- added H105: MountingHole_Pad, MountingHole:MountingHole_3.2mm_M3_DIN965_Pad, F.Cu at (75.4, 123.8)
- added H106: MountingHole_Pad, MountingHole:MountingHole_3.2mm_M3_DIN965_Pad, F.Cu at (75.4, 112.7)
- added J101: Conn_01x05, Connector_PinSocket_2.54mm:PinSocket_1x05_P2.54mm_Horizontal, F.Cu at (122.2, 95.7)
- added J102: Conn_01x05, Connector_PinSocket_2.54mm:PinSocket_1x05_P2.54mm_Horizontal, F.Cu at (112.0, 159.2)
- added J201: Conn_01x03, Connector_PinSocket_2.54mm:PinSocket_1x03_P2.54mm_Vertical, F.Cu at (147.1, 100.6)
- added J202: Conn_01x03, Connector_PinSocket_2.54mm:PinSocket_1x03_P2.54mm_Vertical, F.Cu at (134.6, 100.6)
- added J203: Conn_01x03, Connector_PinSocket_2.54mm:PinSocket_1x03_P2.54mm_Vertical, F.Cu at (129.3, 130.6)
- added J204: Conn_01x03, Connector_PinSocket_2.54mm:PinSocket_1x03_P2.54mm_Vertical, F.Cu at (142.0, 130.8)
- added P101: Conn_01x03_Male, Connector_PinHeader_2.54mm:PinHeader_1x03_P2.54mm_Vertical, F.Cu at (90.5, 152.8)
- added P102: Conn_01x03_Male, Connector_PinHeader_2.54mm:PinHeader_1x03_P2.54mm_Vertical, F.Cu at (95.1, 152.8)
- added P103: Conn_01x03_Male, Connector_PinHeader_2.54mm:PinHeader_1x03_P2.54mm_Vertical, F.Cu at (99.8, 152.8)
- added PM101: Pro_Micro, buttonbox:promicro, F.Cu at (103.0, 118.1)
- added R201: 10k, Resistor_SMD:R_0805_2012Metric_Pad1.15x1.40mm_HandSolder, B.Cu at (142.0, 108.5)
- added R202: 10k, Resistor_SMD:R_0805_2012Metric_Pad1.15x1.40mm_HandSolder, B.Cu at (139.4, 108.5)
- added R203: 10k, Resistor_SMD:R_0805_2012Metric_Pad1.15x1.40mm_HandSolder, B.Cu at (136.9, 108.5)
- added R204: 10k, Resistor_SMD:R_0805_2012Metric_Pad1.15x1.40mm_HandSolder, B.Cu at (134.4, 108.5)
- added R205: 10k, Resistor_SMD:R_0805_2012Metric_Pad1.15x1.40mm_HandSolder, B.Cu at (134.4, 125.0)
- added R206: 10k, Resistor_SMD:R_0805_2012Metric_Pad1.15x1.40mm_HandSolder, B.Cu at (136.9, 125.0)
- added R207: 10k, Resistor_SMD:R_0805_2012Metric_Pad1.15x1.40mm_HandSolder, B.Cu at (139.4, 125.0)
- added R208: 10k, Resistor_SMD:R_0805_2012Metric_Pad1.15x1.40mm_HandSolder, B.Cu at (142.0, 125.0)
- added R301: 10k, Resistor_SMD:R_0805_2012Metric_Pad1.15x1.40mm_HandSolder, F.Cu at (239.1, 130.2)
- added R302: 10k, Resistor_SMD:R_0805_2012Metric_Pad1.15x1.40mm_HandSolder, F.Cu at (179.3, 100.7)
- added R303: 10k, Resistor_SMD:R_0805_2012Metric_Pad1.15x1.40mm_HandSolder, F.Cu at (176.3, 96.1)
- added R304: 10k, Resistor_SMD:R_0805_2012Metric_Pad1.15x1.40mm_HandSolder, F.Cu at (239.1, 125.5)
- added R305: 10k, Resistor_SMD:R_0805_2012Metric_Pad1.15x1.40mm_HandSolder, F.Cu at (231.9, 120.9)
- added R306: 10k, Resistor_SMD:R_0805_2012Metric_Pad1.15x1.40mm_HandSolder, F.Cu at (242.0, 130.2)
- added R307: 10k, Resistor_SMD:R_0805_2012Metric_Pad1.15x1.40mm_HandSolder, F.Cu at (176.3, 100.8)
- added R308: 10k, Resistor_SMD:R_0805_2012Metric_Pad1.15x1.40mm_HandSolder, F.Cu at (173.4, 96.1)
- added SR201: Conn_02x08_Counter_Clockwise, Package_DIP:DIP-16_W7.62mm, F.Cu at (129.3, 120.7)
- added SR301: Conn_02x08_Counter_Clockwise, Package_DIP:DIP-16_W7.62mm, F.Cu at (176.5, 120.7)
Routing:
- net +5V: track 196.9 -> 9.30 mm, vias 4 -> 0
- net /PM_B5: track 84.6 -> 0.00 mm, vias 4 -> 0
- net /PM_B1: track 79.8 -> 0.00 mm, vias 4 -> 0
- net /CT_C_1: track 52.3 -> 0.00 mm
- net /CT_AX_3: track 51.0 -> 0.00 mm
- net /CT_AX_1: track 42.8 -> 0.00 mm
- net /CT_C_3: track 42.3 -> 0.00 mm
- net /CT_R_3: track 38.4 -> 0.00 mm
- net /CT_C_4: track 37.9 -> 0.00 mm, vias 1 -> 0
- net /CT_AX_TRTL: track 35.8 -> 0.00 mm
- net /CT_AX_4: track 33.9 -> 0.00 mm
- net /PM_B3: track 33.5 -> 0.00 mm
- net /CT_AX_2: track 32.6 -> 0.00 mm
- net /SR_QH2: track 27.9 -> 0.00 mm
- net /CT_C_2: track 27.4 -> 0.00 mm
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Other:
- board size 112 x 36.6 mm -> 150 x 72 mm
- board text added: "5V SL CLK DATA GND"
- board text removed: "- AX0 AX1 AX3 C1 C3 R3 R1"
- board text removed: "- AX2 AX4 C4 C2 GND R2 VCC"
- board text removed: "5V SL CLK SER2 GND"
- board text removed: "B2"
- board text removed: "B4"
- board text removed: "B6"
- board text removed: "CT"
- board text removed: "D C B A"
- board text removed: "D2 C2 B2 A2"
- board text removed: "E F G H"
- board text removed: "E2 F2 G2 H2"
- board text removed: "SW3"
