File: box.sch (KiCad schematic (older format))
At the start: 42 parts, among them J1 Conn_01x03, J10 Conn_01x03, J11 Conn_01x05, J2 Conn_01x03, J3 Conn_01x03, J4 Conn_01x03, J5 Conn_01x03, J6 Conn_01x03, J7 Conn_01x03, J8 Conn_01x03, J9 Conn_01x03

Commit message: Update March 21st
Parts:
- removed C2, C3, C4: 470n, Capacitor_SMD:C_0805_2012Metric_Pad1.15x1.40mm_HandSolder, symbol Device:C
- removed CT1: Conn_02x08_Counter_Clockwise, Connector_PinSocket_2.54mm:PinSocket_2x08_P2.54mm_Vertical, symbol Connector_Generic:Conn_02x08_Odd_Even
- removed J1, J10, J2, J3, J4, J5, J6, J7, J8, J9: Conn_01x03, Connector_PinSocket_2.54mm:PinSocket_1x03_P2.54mm_Vertical, symbol Connector_Generic:Conn_01x03
- removed R1, R10, R11, R12, R13, R14, R15, R16, R17, R18, R19, R2, R20, R3, R4, R5, R6, R7, R8, R9: 10k, Resistor_SMD:R_0805_2012Metric_Pad1.15x1.40mm_HandSolder, symbol Device:R
- removed SR1, SR2: Conn_02x08_Counter_Clockwise, Package_DIP:DIP-16_W7.62mm, symbol Connector_Generic:Conn_02x08_Counter_Clockwise
- added C102, C103: 470n, Capacitor_SMD:C_0805_2012Metric_Pad1.15x1.40mm_HandSolder, symbol Device:C
- added H104, H105, H106: MountingHole_Pad, MountingHole:MountingHole_3.2mm_M3_DIN965_Pad, symbol Mechanical:MountingHole_Pad
- added J102: Conn_01x05, Connector_PinSocket_2.54mm:PinSocket_1x05_P2.54mm_Horizontal, symbol Connector_Generic:Conn_01x05
- added P101, P102, P103: Conn_01x03_Male, Connector_PinHeader_2.54mm:PinHeader_1x03_P2.54mm_Vertical, symbol Connector:Conn_01x03_Male
- J101: renamed from J11; footprint Connector_PinSocket_2.54mm:PinSocket_1x05_P2.54mm_Vertical -> Connector_PinSocket_2.54mm:PinSocket_1x05_P2.54mm_Horizontal
- renumbered C1 to C101, H1 to H101, H2 to H102, H3 to H103, PM1 to PM101
Connections:
- net labels added: CAT, H1, H2, H3, H4, H5, H6, H7, JET, SR_QH, THR_L, THR_R, V1, V2, V3, V4, V5, alt_baro, alt_rdr, bearing_left, bearing_right, flaps_dn, flaps_up, form_light, gear_dn, gear_up, hdg_left, hdg_right, hook_dn, hook_up, hud_bright, hud_day, hud_night, hud_norm, hud_rej2, pos_light
- net labels removed: CT_AX_1, CT_AX_2, CT_AX_3, CT_AX_4, CT_AX_TRTL, CT_C_1, CT_C_2, CT_C_3, CT_C_4, CT_R_1, CT_R_2, CT_R_3, CT_VCC, SR_A2, SR_B2, SR_C2, SR_D2, SR_E2, SR_F2, SR_G2, SR_H2, SR_QH1, SR_QH2, SR_QHN1, SR_QHN2, SR_SER1, SW1, SW2, SW3
- wire segments 64 -> 27
Other:
- note added: "B: Push-buttons"
- note added: "Buttons"
- note added: "Buttons:\nH1-H7: horisontal buttons, A/P ... on/off\nV1-V5: vertical buttons, hsel, balt, ralt ..\nThr L, R: throttle to idle\nCAT: Attach catapult\nJET: jettison\n\nToggles:\n- hook up down\n- gear\n- flaps\n- HD1-2: Heading\n- BE1-2: bearing/course\n- HUD day/night: on-on or on-off-on?\n- HUD rej: norm-rej1-rej2\n- ALT: baro-rdr\n\nRotaries:\n- formation light\n- position light\n- ch 1, increas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"
- note added: "J: On-Off-On momentary toggles"
- note added: "Optional: data to the next Shift register"
- note added: "P: Rotaries"
- note added: "Toggles"
- note removed: "CT: Cougar throttle"
- note removed: "Connects to a button matrix \nwith 4 columns and 3 rows"
- note removed: "Flaps"
- note removed: "Gear"
- note removed: "Master arm"
- note removed: "On-Off-On momentary"
- note removed: "SR: Shift register 74HC165"
- note removed: "Toggle 1"
- note removed: "Toggle 2"
- note removed: "Toggle 3"
- note removed: "Toggle 4"
- note removed: "Toggle 5"
- note removed: "Toggle 6"
- note removed: "Toggle 7"
- moved on the sheet: C101, H101, H102, H103, J101
